File: ProgramingAddOn.kicad_pcb (KiCad board)
At the start: 6 copper layers, 37.5 x 48.3 mm, 26 parts, among them J1 USB_B_Mini, J4 Conn_01x12_Male, J5 Conn_01x12_Female, SW1 SW_DIP_x02, SW2 SW_Push, SW3 SW_Push, SW4 SW_Push, SW5 SW_DIP_x04, SW6 SW_Push, SW7 SW_DIP_x04, U1 CP2102N-Axx-xQFN20

Commit message: Update part descriptions. Change USB mini to micro.
Parts:
- J1: value USB_B_Mini -> USB_B_Micro
Changed lines of the file:
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@@
       (effects (font (size 1 1) (thickness 0.15)))
     )
-    (fp_text value "USB_B_Mini" (at 0 4.75 90) (layer "F.Fab")
+    (fp_text value "USB_B_Micro" (at 0 4.75 90) (layer "F.Fab")
       (effects (font (size 1 1) (thickness 0.15)))
     )
